Commit message: add mobile base

File: description/manipulator/urdf/manipulator.urdf.xacro (robot description, xacro)
@@ -4,7 +4,5 @@
     <xacro:arg name="is_sim" default="true"/>
     <!-- Include Gazebo Parameters -->
-    <xacro:include filename="$(find manipulator)/description/urdf/manipulator_gazebo.xacro" />
-    <!-- Include ros2_control Plugins -->
-    <xacro:include filename="$(find manipulator)/description/urdf/ros2_control.xacro" />
+    <xacro:include filename="$(find mobile_bot)/description/manipulator/urdf/manipulator_gazebo.xacro" />
     <!-- Useful XACRO Variables (Properties) -->
     <xacro:property name="PI" value="3.14159265359" />
@@ -31,11 +29,11 @@
     </xacro:macro>
     <!-- Links -->
-    <link name="world"/>
-    <link name="base_link">
+    <!-- <link name="world"/> -->
+    <link name="manipulator_base_link">
         <xacro:default_inertial mass="1.0"/>
         <visual>
             <origin rpy="0 0 0" xyz="-0.5 -0.5 0"/>
             <geometry>
-                <mesh filename="package://manipulator/description/meshes/basement.STL" scale="0.01 0.01 0.01"/>
+                <mesh filename="package://mobile_bot/description/manipulator/meshes/basement.STL" scale="0.01 0.01 0.01"/>
             </geometry>
         </visual>
@@ -43,5 +41,5 @@
             <origin rpy="0 0 0" xyz="-0.5 -0.5 0"/>
             <geometry>
-                <mesh filename="package://manipulator/description/meshes/basement.STL" scale="0.01 0.01 0.01"/>
+                <mesh filename="package://mobile_bot/description/manipulator/meshes/basement.STL" scale="0.01 0.01 0.01"/>
             </geometry>
         </collision>
@@ -52,5 +50,5 @@
             <origin rpy="0 0 0" xyz="-0.39 -0.39 -0.56"/>
             <geometry>
-                <mesh filename="package://manipulator/description/meshes/base_plate.STL" scale="0.01 0.01 0.01"/>
+                <mesh filename="package://mobile_bot/description/manipulator/meshes/base_plate.STL" scale="0.01 0.01 0.01"/>
             </geometry>
         </visual>
@@ -58,5 +56,5 @@
             <origin rpy="0 0 0" xyz="-0.39 -0.39 -0.56"/>
             <geometry>
-                <mesh filename="package://manipulator/description/meshes/base_plate.STL" scale="0.01 0.01 0.01"/>
+                <mesh filename="package://mobile_bot/description/manipulator/meshes/base_plate.STL" scale="0.01 0.01 0.01"/>
             </geometry>
         </collision>
@@ -67,5 +65,5 @@
             <origin rpy=" 0 -${PI / 2} ${PI / 2}" xyz="0.19 0.06 -0.08"/>
             <geometry>
-                <mesh filename="package://manipulator/description/meshes/forward_drive_arm.STL" scale="0.01 0.01 0.01"/>
+                <mesh filename="package://mobile_bot/description/manipulator/meshes/forward_drive_arm.STL" scale="0.01 0.01 0.01"/>
             </geometry>
         </visual>
@@ -73,5 +71,5 @@
             <origin rpy=" 0 -${PI / 2} ${PI / 2}" xyz="0.19 0.06 -0.08"/>
             <geometry>
-                <mesh filename="package://manipulator/description/meshes/forward_drive_arm.STL" scale="0.01 0.01 0.01"/>
+                <mesh filename="package://mobile_bot/description/manipulator/meshes/forward_drive_arm.STL" scale="0.01 0.01 0.01"/>
             </geometry>
         </collision>
@@ -82,5 +80,5 @@
             <origin rpy="${PI / 2} 0 ${PI / 2}" xyz="-0.03 -0.4 -0.06"/>
             <geometry>
-                <mesh filename="package://manipulator/description/meshes/horizontal_arm.STL" scale="0.01 0.01 0.01"/>
+                <mesh filename="package://mobile_bot/description/manipulator/meshes/horizontal_arm.STL" scale="0.01 0.01 0.01"/>
             </geometry>
         </visual>
@@ -88,5 +86,5 @@
             <origin rpy="${PI / 2} 0 ${PI / 2}" xyz="-0.03 -0.4 -0.06"/>
             <geometry>
-                <mesh filename="package://manipulator/description/meshes/horizontal_arm.STL" scale="0.01 0.01 0.01"/>
+                <mesh filename="package://mobile_bot/description/manipulator/meshes/horizontal_arm.STL" scale="0.01 0.01 0.01"/>
             </geometry>
         </collision>
@@ -97,5 +95,5 @@
             <origin rpy="0 0 ${PI / 2}" xyz="0 -0.05 -0.15"/>
             <geometry>
-                <mesh filename="package://manipulator/description/meshes/claw_support.STL" scale="0.01 0.01 0.01"/>
+                <mesh filename="package://mobile_bot/description/manipulator/meshes/claw_support.STL" scale="0.01 0.01 0.01"/>
             </geometry>
         </visual>
@@ -103,5 +101,5 @@
             <origin rpy="0 0 ${PI / 2}" xyz="0 -0.05 -0.15"/>
             <geometry>
-                <mesh filename="package://manipulator/description/meshes/claw_support.STL" scale="0.01 0.01 0.01"/>
+                <mesh filename="package://mobile_bot/description/manipulator/meshes/claw_support.STL" scale="0.01 0.01 0.01"/>
             </geometry>
         </collision>
@@ -112,5 +110,5 @@
             <origin rpy="0 0 -${PI / 2}" xyz="-0.1 0.50 -0.1"/>
             <geometry>
-                <mesh filename="package://manipulator/description/meshes/right_finger.STL" scale="0.01 0.01 0.01"/>
+                <mesh filename="package://mobile_bot/description/manipulator/meshes/right_finger.STL" scale="0.01 0.01 0.01"/>
             </geometry>
         </visual>
@@ -118,5 +116,5 @@
             <origin rpy="0 0 -${PI / 2}" xyz="-0.1 0.50 -0.1"/>
             <geometry>
-                <mesh filename="package://manipulator/description/meshes/right_finger.STL" scale="0.01 0.01 0.01"/>
+                <mesh filename="package://mobile_bot/description/manipulator/meshes/right_finger.STL" scale="0.01 0.01 0.01"/>
             </geometry>
         </collision>
@@ -127,5 +125,5 @@
             <origin rpy="0 0 -${PI / 2}" xyz="-0.04 0.50 -0.1"/>
             <geometry>
-                <mesh filename="package://manipulator/description/meshes/left_finger.STL" scale="0.01 0.01 0.01"/>
+                <mesh filename="package://mobile_bot/description/manipulator/meshes/left_finger.STL" scale="0.01 0.01 0.01"/>
             </geometry>
         </visual>
@@ -133,5 +131,5 @@
             <origin rpy="0 0 -${PI / 2}" xyz="-0.04 0.50 -0.1"/>
             <geometry>
-                <mesh filename="package://manipulator/description/meshes/left_finger.STL" scale="0.01 0.01 0.01"/>
+                <mesh filename="package://mobile_bot/description/manipulator/meshes/left_finger.STL" scale="0.01 0.01 0.01"/>
             </geometry>
         </collision>
@@ -142,5 +140,5 @@
             <origin rpy="-1.57 0 -1.57" xyz="-0.1 0.125 0.15"/>
             <geometry>
-                <mesh filename="package://manipulator/description/meshes/pi_camera.STL" scale="0.01 0.01 0.01"/>
+                <mesh filename="package://mobile_bot/description/manipulator/meshes/pi_camera.STL" scale="0.01 0.01 0.01"/>
             </geometry>
         </visual>
@@ -148,16 +146,10 @@
             <origin rpy="-1.57 0 -1.57" xyz="-0.1 0.125 0.15"/>
             <geometry>
-                <mesh filename="package://manipulator/description/meshes/pi_camera.STL" scale="0.01 0.01 0.01"/>
-            </geometry>
-        </collision>
-    </link>
-    <!-- Joints -->
-    <joint name="virtual_joint" type="fixed">
-        <parent link="world"/>
-        <child link="base_link"/>
-        <origin xyz="0 0 0" rpy="0 0 0"/>
-    </joint>
+                <mesh filename="package://mobile_bot/description/manipulator/meshes/pi_camera.STL" scale="0.01 0.01 0.01"/>
+            </geometry>
+        </collision>
+    </link>
     <joint name ="joint_1" type="revolute">
-        <parent link="base_link"/>
+        <parent link="manipulator_base_link"/>
         <child link = "base_plate"/>
         <origin xyz="0 0 0.307"/>
@@ -205,5 +197,5 @@
     </joint>
     <joint name ="rgb_camera_joint" type="fixed">
-        <parent link="base_link"/>
+        <parent link="manipulator_base_link"/>
         <child link = "rgb_camera"/>
         <origin xyz="0 0.45 0.2" rpy="0 -0.5 1.57"/>

File: description/manipulator/urdf/manipulator_gazebo.xacro (robot description, xacro)
@@ -6,5 +6,5 @@
         <robot_param>robot_description</robot_param>
         <robot_param_node>robot_state_publisher</robot_param_node>
-        <parameters>$(find manipulator)/config/ros2_control_params.yaml</parameters>
+        <parameters>$(find mobile_bot)/config/ros2_control_params.yaml</parameters>
       </plugin>
     </gazebo>
