Commit message: tune omni movement jerk

File: description/omni_urdf/wheel/wheel_100mm_light.urdf.xacro (robot description, xacro)
@@ -22,5 +22,5 @@
       <visual>
         <geometry>
-          <cylinder length="0.040" radius="0.15" />
+          <cylinder length="0.1" radius="0.15" />
         </geometry>
         <origin xyz="0 0 0" rpy="0 0 0"/>
@@ -29,5 +29,5 @@
       <collision>
         <geometry>
-          <cylinder length="0.040" radius="0.15" />
+          <cylinder length="0.1" radius="0.15" />
         </geometry>
         <origin xyz="0 0 0" rpy="0 0 0"/>
@@ -35,5 +35,5 @@
       </collision>
       <inertial>
-        <mass value="1.288"/>
+        <mass value="3.5"/>
         <inertia ixx="0.00235" ixy="0" ixz="0" iyy="0.00235" iyz="0" izz="0.00004"/>
       </inertial>
@@ -42,5 +42,5 @@
       <material>Gazebo/Gray</material>
       <mu1>0.8</mu1>
-      <mu2>0.05</mu2>
+      <mu2>0.1</mu2>
       <fdir1>0 1.0 0</fdir1>
       <kp value="30000000.0" />

Commit message: rotate manipulator to face forward

File: description/omni_urdf/wheel/wheel_100mm_light.urdf.xacro (robot description, xacro)
@@ -41,5 +41,5 @@
     <gazebo reference="${prefix}_housing_link">
       <material>Gazebo/Gray</material>
-      <mu1>0.8</mu1>
+      <mu1>0.9</mu1>
       <mu2>0.1</mu2>
       <fdir1>0 1.0 0</fdir1>

File: description/robot.urdf.xacro (robot description, xacro)
@@ -68,5 +68,5 @@
         <parent link="omnibot_base_link" />
         <child link="manipulator_base_link" />
-        <origin xyz="0 0 0.1" rpy="0 0 0" />
+        <origin xyz="0 0 0.1" rpy="0 0 ${pi/2}" />
     </joint>
     <xacro:omnibot_gazebo prefix="" />
