Commit message: reconfigure workspace

File: manipulator_description/description/manipulator/urdf/manipulator_gazebo.xacro (robot description, xacro)
@@ -6,5 +6,5 @@
         <robot_param>robot_description</robot_param>
         <robot_param_node>robot_state_publisher</robot_param_node>
-        <parameters>$(find mobile_bot)/config/ros2_control_params.yaml</parameters>
+        <parameters>$(find manipulator_description)/config/ros2_control_params.yaml</parameters>
       </plugin>
     </gazebo>

File: manipulator_description/description/omni_urdf/base/base.urdf.xacro (robot description, xacro)
@@ -1,5 +1,5 @@
 <?xml version="1.0"?>
 <robot xmlns:xacro="http://ros.org/wiki/xacro">
-  <xacro:include filename="$(find mobile_bot)/description/omni_urdf/base/base.gazebo.xacro" />
+  <xacro:include filename="$(find manipulator_description)/description/omni_urdf/base/base.gazebo.xacro" />
   <xacro:property name="base_length" value="1.5" />
   <xacro:property name="base_height" value="0.1" />

File: manipulator_description/description/omni_urdf/wheel/wheel.urdf.xacro (robot description, xacro)
@@ -12,5 +12,5 @@
       <visual>
         <geometry>
-          <mesh filename="file://$(find mobile_bot)/description/omni_urdf/STL/omni_barrel.stl" />
+          <mesh filename="file://$(find manipulator_description)/description/omni_urdf/STL/omni_barrel.stl" />
         </geometry>
         <material name="black"/>
@@ -18,5 +18,5 @@
       <collision>
         <geometry>
-          <mesh filename="file://$(find mobile_bot)/description/omni_urdf/STL/omni_barrel.stl" />
+          <mesh filename="file://$(find manipulator_description)/description/omni_urdf/STL/omni_barrel.stl" />
         </geometry>
       </collision>
@@ -65,5 +65,5 @@
       <visual>
         <geometry>
-          <mesh filename="file://$(find mobile_bot)/description/omni_urdf/STL/omni_housing.stl" />
+          <mesh filename="file://$(find manipulator_description)/description/omni_urdf/STL/omni_housing.stl" />
         </geometry>
         <origin xyz="0 0 0" rpy="0 0 0"/>

File: manipulator_description/description/omni_urdf/wheel/wheel_100mm.urdf.xacro (robot description, xacro)
@@ -12,5 +12,5 @@
       <visual>
         <geometry>
-          <mesh filename="file://$(find mobile_bot)/description/omni_urdf/STL/omni_barrel_100mm.stl" />
+          <mesh filename="file://$(find manipulator_description)/description/omni_urdf/STL/omni_barrel_100mm.stl" />
         </geometry>
         <material name="black"/>
@@ -18,5 +18,5 @@
       <collision>
         <geometry>
-          <mesh filename="file://$(find mobile_bot)/description/omni_urdf/STL/omni_barrel_100mm.stl" />
+          <mesh filename="file://$(find manipulator_description)/description/omni_urdf/STL/omni_barrel_100mm.stl" />
         </geometry>
       </collision>
@@ -65,5 +65,5 @@
       <visual>
         <geometry>
-          <mesh filename="file://$(find mobile_bot)/description/omni_urdf/STL/omni_housing_100mm.stl" />
+          <mesh filename="file://$(find manipulator_description)/description/omni_urdf/STL/omni_housing_100mm.stl" />
         </geometry>
         <origin xyz="0 0 0" rpy="0 0 0"/>
